File: GreenHouse/Incubator/serre light v1.brd (EAGLE design)
At the start: 400 x 325 mm, 74 parts, among them IC1 TPS54201, IC2 TPS54201, IC3 TPS54201, IC5 TPS54201, J3 CON-MICROFIT-1X2, J4 CON-MICROFIT-1X2

Commit message: Incubator working firmware
Parts:
- moved R3 0.79 mm to (19.5, 66.0)
- moved C8 0.58 mm to (18.5, 68.8)
Routing:
- net N$19: track 3.51 -> 4.19 mm
Changed lines of the file:
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@@
 <setting verticaltext="up"/>
 </settings>
-<grid distance="0.25" unitdist="mm" unit="mm" style="lines" multiple="1" display="yes" altdistance="0.025" altunitdist="inch" altunit="inch"/>
+<grid distance="0.25" unitdist="mm" unit="mm" style="lines" multiple="1" display="yes" altdistance="0.01" altunitdist="mm" altunit="mm"/>
 <layers>
 <layer number="1" name="Top" color="4" fill="1" visible="yes" active="yes"/>
@@
 <layer number="23" name="tOrigins" color="15" fill="1" visible="yes" active="yes"/>
 <layer number="24" name="bOrigins" color="15" fill="1" visible="yes" active="yes"/>
-<layer number="25" name="tNames" color="7" fill="1" visible="no" active="yes"/>
+<layer number="25" name="tNames" color="7" fill="1" visible="yes" active="yes"/>
 <layer number="26" name="bNames" color="7" fill="1" visible="no" active="yes"/>
-<layer number="27" name="tValues" color="7" fill="1" visible="no" active="yes"/>
+<layer number="27" name="tValues" color="7" fill="1" visible="yes" active="yes"/>
 <layer number="28" name="bValues" color="7" fill="1" visible="no" active="yes"/>
-<layer number="29" name="tStop" color="7" fill="3" visible="no" active="yes"/>
+<layer number="29" name="tStop" color="7" fill="3" visible="yes" active="yes"/>
 <layer number="30" name="bStop" color="7" fill="6" visible="no" active="yes"/>
 <layer number="31" name="tCream" color="7" fill="4" visible="no" active="yes"/>
@@
 <attribute name="VALUE" x="31.5275" y="52.585" size="1.27" layer="27" rot="R270"/>
 </element>
-<element name="R3" library="Bonelli" package="R0805" value="1.2k" x="19.7325" y="66.715" smashed="yes" rot="R270">
-<attribute name="NAME" x="20.6325" y="68.015" size="0.5" layer="25" rot="R270"/>
-<attribute name="VALUE" x="18.3325" y="68.015" size="0.5" layer="27" rot="R270"/>
+<element name="R3" library="Bonelli" package="R0805" value="1.2k" x="19.4825" y="65.965" smashed="yes" rot="R270">
+<attribute name="NAME" x="20.3825" y="67.265" size="0.5" layer="25" rot="R270"/>
+<attribute name="VALUE" x="18.0825" y="67.265" size="0.5" layer="27" rot="R270"/>
 </element>
 <element name="IC2" library="Bonelli" package="SOT23-6" value="TPS54201" x="21.11" y="71.97" smashed="yes" rot="R180">
@@
 <attribute name="VALUE" x="23.015" y="75.145" size="1.27" layer="27" rot="R180"/>
 </element>
-<element name="C8" library="Bonelli" package="C0603" value="33n" x="18.9825" y="69.0925" smashed="yes" rot="R180">
-<attribute name="NAME" x="20.2825" y="68.383" size="0.5" layer="25" rot="R180"/>
-<attribute name="VALUE" x="20.2825" y="70.302" size="0.5" layer="27" rot="R180"/>
+<element name="C8" library="Bonelli" package="C0603" value="33n" x="18.5025" y="68.7625" smashed="yes" rot="R180">
+<attribute name="NAME" x="19.8025" y="68.053" size="0.5" layer="25" rot="R180"/>
+<attribute name="VALUE" x="19.8025" y="69.972" size="0.5" layer="27" rot="R180"/>
 </element>
 <element name="C9" library="Bonelli" package="C0603" value="100n" x="23.09" y="66.1675" smashed="yes" rot="R180">
@@
 <polygon width="0.3" layer="1" isolate="0.3" thermals="no">
 <vertex x="7.61" y="72.595"/>
-<vertex x="7.61" y="68.72"/>
-<vertex x="18.61" y="68.72"/>
+<vertex x="7.61" y="68.26"/>
+<vertex x="18.61" y="68.26"/>
 <vertex x="18.61" y="71.595"/>
 <vertex x="22.735" y="71.595"/>
@@
 <contactref element="IC2" pad="4"/>
 <contactref element="C8" pad="1"/>
-<wire x1="20.16" y1="70.67" x2="20.16" y2="69.0925" width="0.3" layer="1"/>
-<wire x1="20.16" y1="69.0925" x2="19.8715" y2="69.0925" width="0.3" layer="1"/>
-<wire x1="19.8715" y1="69.0925" x2="19.8715" y2="67.59" width="0.3" layer="1"/>
-<wire x1="19.8715" y1="67.59" x2="19.7325" y2="67.59" width="0.3" layer="1"/>
+<wire x1="20.16" y1="70.67" x2="20.16" y2="70.035" width="0.3" layer="1"/>
+<wire x1="20.16" y1="70.035" x2="19.66" y2="69.535" width="0.3" layer="1"/>
+<wire x1="19.66" y1="69.535" x2="19.66" y2="69.031" width="0.3" layer="1"/>
+<wire x1="19.66" y1="69.031" x2="19.3915" y2="68.7625" width="0.3" layer="1"/>
+<wire x1="19.3915" y1="68.7625" x2="19.3915" y2="66.931" width="0.3" layer="1"/>
+<wire x1="19.4825" y1="66.84" x2="19.3915" y2="66.931" width="0.3" layer="1"/>
 </signal>
 <signal name="N$22">
@@
 <vertex x="24.6" y="71"/>
 </polygon>
-<wire x1="19.7325" y1="65.84" x2="19.865" y2="65.84" width="0.3" layer="1"/>
-<wire x1="19.865" y1="65.84" x2="20.61" y2="65.095" width="0.3" layer="1"/>
-<wire x1="20.61" y1="65.095" x2="25.735" y2="65.095" width="0.3" layer="1"/>
+<wire x1="25.735" y1="65.095" x2="19.4875" y2="65.095" width="0.3" layer="1"/>
+<wire x1="19.4825" y1="65.09" x2="19.4875" y2="65.095" width="0.3" layer="1"/>
 <wire x1="25.735" y1="65.095" x2="26.235" y2="65.595" width="0.3" layer="1"/>
 <wire x1="26.235" y1="65.595" x2="26.235" y2="68.1455" width="0.3" layer="1"/>
@@
 <contactref element="J2" pad="4"/>
 <wire x1="23.5" y1="125.81" x2="22.29" y2="127.02" width="0.3" layer="1"/>
-<wire x1="21.11" y1="70.67" x2="21.125" y2="70.655" width="0.3" layer="1"/>
-<wire x1="21.125" y1="70.655" x2="21.125" y2="68.5" width="0.3" layer="1"/>
-<via x="21.125" y="68.5" extent="1-16" drill="0.8" diameter="1.6"/>
-<wire x1="21.125" y1="68.5" x2="21.125" y2="65.675" width="0.3" layer="16"/>
-<wire x1="21.125" y1="65.675" x2="21.925" y2="64.875" width="0.3" layer="16"/>
+<wire x1="21.11" y1="70.67" x2="20.955" y2="70.515" width="0.3" layer="1"/>
+<wire x1="20.955" y1="70.515" x2="20.955" y2="68.29" width="0.3" layer="1"/>
+<via x="20.955" y="68.29" extent="1-16" drill="0.8" diameter="1.6"/>
+<wire x1="20.955" y1="68.29" x2="20.955" y2="65.845" width="0.3" layer="16"/>
+<wire x1="20.955" y1="65.845" x2="21.925" y2="64.875" width="0.3" layer="16"/>
 <wire x1="21.925" y1="64.875" x2="26.075" y2="64.875" width="0.3" layer="16"/>
 <wire x1="26.075" y1="64.875" x2="26.875" y2="65.675" width="0.3" layer="16"/>
